Commit message: Ported same inertial parameters into left hand xacro.

File: allegro_hand_description/allegro_hand_description_left.xacro (robot description, xacro)
@@ -45,4 +45,10 @@
     <xacro:property name="limit_3_t_low" value="-0.262"/>
     <!-- ============================================================================= -->
+    <!-- Used for fixing robot to Gazebo 'base_link' -->
+    <link name="world"/>
+    <joint name="fixed" type="fixed">
+      <parent link="world"/>
+      <child link="base_link"/>
+    </joint>
     <!-- BASE -->
     <link name="base_link">
@@ -62,4 +68,12 @@
             </geometry>
         </collision>
+        <inertial>
+          <origin xyz="0 0 ${base_link_z/2}" rpy="0 0 0"/>
+          <mass value="0.4154"/>
+          <inertia
+              ixx="1e-4" ixy="0.0" ixz="0.0"
+              iyy="1e-4" iyz="0.0"
+              izz="1e-4"/>
+        </inertial>
     </link>
     <!-- ============================================================================= -->
@@ -120,8 +134,15 @@
                         xyz="${-0.0358/2+0.0} ${-.018/2} ${.029/2}"/>
             </collision>
+            <inertial>
+              <mass value="0.0176" />
+              <origin xyz="0 0 0" rpy="0 0 0"/>
+              <inertia ixx="1.89273333333e-5" ixy="7.16716e-06" ixz="5.35568e-06"
+                       iyy="1.43008213333e-05" iyz="6.8068e-06"
+                       izz="1.89273333333e-05" />
+            </inertial>
         </link>
         <joint name="joint_${finger_num*4+0}" type="revolute">
             <axis xyz="+1 0 0"/>
-            <limit effort="0" velocity="0"
+            <limit effort="15" velocity="7"
                    lower="${limit_0_t_low-joint_safety_margin}"
                    upper="${limit_0_t_up-joint_safety_margin}"/>
@@ -130,4 +151,5 @@
             <origin rpy="${finger_angle_r} ${finger_angle_p} ${finger_angle_y}"
                     xyz="${offset_origin_x} ${offset_origin_y} ${offset_origin_z}"/>
+            <dynamics damping="3" friction="10"/>
         </joint>
         <!-- [LINK 13] -->
@@ -147,8 +169,15 @@
                 <origin rpy="0 0 0" xyz="0 0 ${link1_t_z/2}"/>
             </collision>
+            <inertial>
+              <mass value="0.0119" />
+              <origin xyz="0 0 0" rpy="0 0 0"/>
+              <inertia ixx="4.24250866667e-06" ixy="1.032087e-06" ixz="1.603525e-06"
+                       iyy="4.52362633333e-06" iyz="1.44808125e-06"
+                       izz="4.24250866667e-06" />
+            </inertial>
         </link>
         <joint name="joint_${finger_num*4+1}" type="revolute">
             <axis xyz="0 0 -1"/>
-            <limit effort="0" velocity="0"
+            <limit effort="15" velocity="7"
                    lower="${limit_1_t_low+joint_safety_margin}"
                    upper="${limit_1_t_up-joint_safety_margin}"/>
@@ -156,4 +185,5 @@
             <child link="link_${finger_num*4+1}"/>
             <origin xyz="-0.027 -0.005 0.0399"/>
+			<dynamics damping="3" friction="5"/>
         </joint>
         <!-- [LINK 14] -->
@@ -172,8 +202,14 @@
                 <origin rpy="0 0 0" xyz="0 0 ${link2_t_z/2}"/>
             </collision>
+            <inertial>
+              <mass value="0.038" />
+              <origin xyz="0 0 0" rpy="0 0 0"/>
+              <inertia ixx="4.30439933333e-05" ixy="9.57068e-06" ixz="5.1205e-06" iyy="1.44451933333e-05"
+                       iyz="1.342825e-05" izz="4.30439933333e-05" />
+            </inertial>
         </link>
         <joint name="joint_${finger_num*4+2}" type="revolute">
             <axis xyz="0 1 0"/>
-            <limit effort="0" velocity="0"
+            <limit effort="15" velocity="7"
                    lower="${limit_2_t_low+joint_safety_margin}"
                    upper="${limit_2_t_up-joint_safety_margin}"/>
@@ -181,4 +217,5 @@
             <child link="link_${finger_num*4+2}"/>
             <origin xyz="0 0 ${link1_t_z}"/>
+            <dynamics damping="3" friction="10"/>
         </joint>
         <!-- [LINK 15] -->
@@ -197,8 +234,15 @@
                 <origin rpy="0 0 0" xyz="0 0 ${(link3_t_z-fingerTip_r)/2}"/>
             </collision>
+            <inertial>
+              <mass value="0.0388" />
+              <origin xyz="0 0 0" rpy="0 0 0"/>
+              <inertia ixx="3.29223173333e-05" ixy="8.042076e-06" ixz="5.2283e-06"
+                       iyy="1.47493026667e-5" iyz="1.1283525e-5"
+                       izz="3.29223173333e-05" />
+            </inertial>
         </link>
         <joint name="joint_${finger_num*4+3}" type="revolute">
             <axis xyz="0 1 0"/>
-            <limit effort="0" velocity="0"
+            <limit effort="15" velocity="7"
                    lower="${limit_3_t_low+joint_safety_margin}"
                    upper="${limit_3_t_up-joint_safety_margin}"/>
@@ -206,4 +250,5 @@
             <child link="link_${finger_num*4+3}"/>
             <origin xyz="0 0 ${link2_t_z}"/>
+            <dynamics damping="3" friction="12"/>
         </joint>
         <!-- [FINGER TIP] -->
@@ -223,4 +268,11 @@
                 <origin rpy="0 0 0" xyz="0 0 0"/>
             </collision>
+            <inertial>
+              <mass value="0.0168" />
+              <origin xyz="0 0 0" rpy="0 0 0"/>
+              <inertia ixx="9.68e-07" ixy="0" ixz="0"
+                       iyy="9.68e-07" iyz="0"
+                       izz="9.68e-07" />
+            </inertial>
         </link>
         <joint name="joint_${finger_num*4+3}_tip" type="fixed">
@@ -248,8 +300,15 @@
                 <origin rpy="0 0 0" xyz="0 0 ${link0_z/2}"/>
             </collision>
+            <inertial>
+              <mass value="0.0119" />
+              <origin xyz="0 0 0" rpy="0 0 0"/>
+              <inertia ixx="1.01666658333e-06" ixy="0.0" ixz="0.0"
+                       iyy="6.47677333333e-07" iyz="0.0"
+                       izz="1.01666658333e-06" />
+            </inertial>
         </link>
         <joint name="joint_${finger_num*4+0}" type="revolute">
             <axis xyz="0 0 1"/>
-            <limit effort="0" velocity="0"
+            <limit effort="15" velocity="7"
                    lower="${limit_0_low+joint_safety_margin}"
                    upper="${limit_0_up-joint_safety_margin}"/>
@@ -258,4 +317,5 @@
             <origin rpy="${finger_angle_r} 0 0"
                     xyz="${offset_origin_x} ${offset_origin_y} ${offset_origin_z}"/>
+            <dynamics damping="3" friction="10"/>
         </joint>
         <!-- [LINK 1, 5, 9] -->
@@ -273,7 +333,14 @@
                 <origin rpy="0 0 0" xyz="0 0 ${link1_z/2}"/>
             </collision>
+            <inertial>
+              <mass value="0.065" />
+              <origin xyz="0 0 0" rpy="0 0 0"/>
+              <inertia ixx="7.95654166667e-05" ixy="1.7199e-05" ixz="8.75875e-06"
+                       iyy="2.47088833333e-05" iyz="2.413125e-05"
+                       izz="7.95654166667e-05" />
+            </inertial>
         </link>
         <joint name="joint_${finger_num*4+1}" type="revolute">
-            <limit effort="0" velocity="0"
+            <limit effort="15" velocity="7"
                    lower="${limit_1_low+joint_safety_margin}"
                    upper="${limit_1_up-joint_safety_margin}"/>
@@ -282,4 +349,5 @@
             <child link="link_${finger_num*4+1}"/>
             <origin xyz="0 0 ${link0_z}"/>
+            <dynamics damping="3" friction="5"/>
         </joint>
         <!-- [LINK 2, 6, 10]-->
@@ -297,8 +365,15 @@
                 <origin rpy="0 0 0" xyz="0 0 ${link2_z/2}"/>
             </collision>
+            <inertial>
+              <mass value="0.0355" />
+              <origin xyz="0 0 0" rpy="0 0 0"/>
+              <inertia ixx="2.63979183333e-05" ixy="6.67968e-06" ixz="4.783625e-06"
+                       iyy="1.34948516667e-05" iyz="9.372e-06"
+                       izz="2.63979183333e-05" />
+            </inertial>
         </link>
         <joint name="joint_${finger_num*4+2}" type="revolute">
             <axis xyz="0 1 0"/>
-            <limit effort="0" velocity="0"
+            <limit effort="15" velocity="7"
                    lower="${limit_2_low+joint_safety_margin}"
                    upper="${limit_2_up-joint_safety_margin}"/>
@@ -306,4 +381,5 @@
             <child link="link_${finger_num*4+2}"/>
             <origin xyz="0 0 ${link1_z}"/>
+            <dynamics damping="8" friction="10"/>
         </joint>
         <!-- [LINK 3, 7, 11] -->
@@ -321,8 +397,15 @@
                 <origin rpy="0 0 0" xyz="0 0 ${(link3_z-fingerTip_r)/2}"/>
             </collision>
+            <inertial>
+              <mass value="0.0096" />
+              <origin xyz="0 0 0" rpy="0 0 0"/>
+              <inertia ixx="4.701248e-06" ixy="1.255968e-06" ixz="1.2936e-06"
+                       iyy="3.649312e-06" iyz="1.7622e-06"
+                       izz="4.701248e-06" />
+            </inertial>
         </link>
         <joint name="joint_${finger_num*4+3}" type="revolute">
             <axis xyz="0 1 0"/>
-            <limit effort="0" velocity="0"
+            <limit effort="15" velocity="7"
                    lower="${limit_3_low+joint_safety_margin}"
                    upper="${limit_3_up-joint_safety_margin}"/>
@@ -330,4 +413,5 @@
             <child link="link_${finger_num*4+3}"/>
             <origin xyz="0 0 ${link2_z}"/>
+            <dynamics damping="10" friction="12"/>
         </joint>
         <!-- [FINGER TIP] -->
@@ -346,4 +430,11 @@
                 </geometry>
             </collision>
+            <inertial>
+              <mass value="0.0168" />
+              <origin xyz="0 0 0" rpy="0 0 0"/>
+              <inertia ixx="9.68e-07" ixy="0" ixz="0"
+                       iyy="9.68e-07" iyz="0"
+                       izz="9.68e-07" />
+            </inertial>
         </link>
         <joint name="joint_${finger_num*4+3}_tip" type="fixed">

File: allegro_hand_description/allegro_hand_description_right.xacro (robot description, xacro)
@@ -125,4 +125,5 @@
                     <color rgba=".2 .2 .2 1"/>
                 </material>
+                <origin rpy="${180*DEG2RAD} 0 0" xyz="0 0 0"/>
             </visual>
             <collision>

Commit message: Renamed base_link -> palm_link.

File: allegro_hand_description/allegro_hand_description_left.xacro (robot description, xacro)
@@ -3,5 +3,5 @@
     <xacro:property name="DEG2RAD" value="0.01745329251"/>
     <!-- ======================== BASE PARAMS ========================= -->
-    <xacro:property name="base_link_z" value="0.095"/>
+    <xacro:property name="palm_link_z" value="0.095"/>
     <!-- ======================== FINGER PARAMS ======================== -->
     <xacro:property name="links_x" value="0.0196"/>
@@ -45,12 +45,6 @@
     <xacro:property name="limit_3_t_low" value="-0.262"/>
     <!-- ============================================================================= -->
-    <!-- Used for fixing robot to Gazebo 'base_link' -->
-    <link name="world"/>
-    <joint name="fixed" type="fixed">
-      <parent link="world"/>
-      <child link="base_link"/>
-    </joint>
-    <!-- BASE -->
-    <link name="base_link">
+    <!-- PALM -->
+    <link name="palm_link">
         <visual>
             <geometry>
@@ -63,11 +57,11 @@
         </visual>
         <collision>
-            <origin rpy="0 0 0" xyz="-0.009300 0 -${base_link_z/2}"/>
+            <origin rpy="0 0 0" xyz="-0.009300 0 -${palm_link_z/2}"/>
             <geometry>
-                <box size="0.0408 0.1130 ${base_link_z}"/>
+                <box size="0.0408 0.1130 ${palm_link_z}"/>
             </geometry>
         </collision>
         <inertial>
-          <origin xyz="0 0 ${base_link_z/2}" rpy="0 0 0"/>
+          <origin xyz="0 0 ${palm_link_z/2}" rpy="0 0 0"/>
           <mass value="0.4154"/>
           <inertia
@@ -147,5 +141,5 @@
                    lower="${limit_0_t_low-joint_safety_margin}"
                    upper="${limit_0_t_up-joint_safety_margin}"/>
-            <parent link="base_link"/>
+            <parent link="palm_link"/>
             <child link="link_${finger_num*4+0}"/>
             <origin rpy="${finger_angle_r} ${finger_angle_p} ${finger_angle_y}"
@@ -313,5 +307,5 @@
                    lower="${limit_0_low+joint_safety_margin}"
                    upper="${limit_0_up-joint_safety_margin}"/>
-            <parent link="base_link"/>
+            <parent link="palm_link"/>
             <child link="link_${finger_num*4+0}"/>
             <origin rpy="${finger_angle_r} 0 0"

File: allegro_hand_description/allegro_hand_description_right.xacro (robot description, xacro)
@@ -3,5 +3,5 @@
     <xacro:property name="DEG2RAD" value="0.01745329251"/>
     <!-- ======================== BASE PARAMS ========================= -->
-    <xacro:property name="base_link_z" value="0.095"/>
+    <xacro:property name="palm_link_z" value="0.095"/>
     <!-- ======================== FINGER PARAMS ======================== -->
     <xacro:property name="links_x" value="0.0196"/>
@@ -45,12 +45,6 @@
     <xacro:property name="limit_3_t_low" value="-0.262"/>
     <!-- ============================================================================= -->
-    <!-- Used for fixing robot to Gazebo 'base_link' -->
-    <link name="world"/>
-    <joint name="fixed" type="fixed">
-      <parent link="world"/>
-      <child link="base_link"/>
-    </joint>
-    <!-- BASE -->
-    <link name="base_link">
+    <!-- PALM -->
+    <link name="palm_link">
         <visual>
             <geometry>
@@ -63,11 +57,11 @@
         </visual>
         <collision>
-            <origin rpy="0 0 0" xyz="-0.009300 0 -${base_link_z/2}"/>
+            <origin rpy="0 0 0" xyz="-0.009300 0 -${palm_link_z/2}"/>
             <geometry>
-                <box size="0.0408 0.1130 ${base_link_z}"/>
+                <box size="0.0408 0.1130 ${palm_link_z}"/>
             </geometry>
         </collision>
         <inertial>
-          <origin xyz="0 0 ${base_link_z/2}" rpy="0 0 0"/>
+          <origin xyz="0 0 ${palm_link_z/2}" rpy="0 0 0"/>
           <mass value="0.4154"/>
           <inertia
@@ -146,5 +140,5 @@
                    lower="${limit_0_t_low-joint_safety_margin}"
                    upper="${limit_0_t_up-joint_safety_margin}"/>
-            <parent link="base_link"/>
+            <parent link="palm_link"/>
             <child link="link_${finger_num*4+0}"/>
             <origin rpy="${finger_angle_r} ${finger_angle_p} ${finger_angle_y}"
@@ -312,5 +306,5 @@
                    lower="${limit_0_low+joint_safety_margin}"
                    upper="${limit_0_up-joint_safety_margin}"/>
-            <parent link="base_link"/>
+            <parent link="palm_link"/>
             <child link="link_${finger_num*4+0}"/>
             <origin rpy="${finger_angle_r} 0 0"

Commit message: Adds a base link as the root, so that the hand is above the origin.

File: allegro_hand_description/allegro_hand_description_left.xacro (robot description, xacro)
@@ -45,4 +45,13 @@
     <xacro:property name="limit_3_t_low" value="-0.262"/>
     <!-- ============================================================================= -->
+    <!-- Base link -->
+    <link name="hand_root">
+      <origin xyz="0 0 0"/>
+    </link>
+    <joint name="root_to_base" type="fixed">
+      <parent link="hand_root"/>
+      <child link="palm_link"/>
+      <origin xyz="0 0 ${palm_link_z}"/>
+    </joint>
     <!-- PALM -->
     <link name="palm_link">
